Commit message: Add pingpong Paddle URDF

File: src/g1_description/urdf/g1_29dof.urdf (robot description, URDF)
Before this commit: robot g1_29dof, 40 links, 39 joints
Links:
- added link pingpong_racket, mass 0.15; collision box size=0.25 0.15 0.02; visual mesh filename=package://g1_description/meshes/Pingpong_paddle_v1_L3.obj scale=0.01 0.01 0.01
Joints:
- added joint racket_fixed_joint: type fixed, parent right_rubber_hand, child pingpong_racket, origin xyz=-0.05 0.00 0.02 rpy=0 -1.57 0

Commit message: hips dont lie

File: src/g1_description/urdf/g1_29dof.urdf (robot description, URDF)
Before this commit: robot g1_29dof, 41 links, 40 joints
Joints:
- joint racket_fixed_joint: origin xyz=-0.05 0.00 0.02 rpy=0 -1.57 0 -> xyz=0.0 0.02 0.02 rpy=1.57 -1.57 1.57
